Commit message: Star Wars agents

File: fcu_sim/urdf/junker/junker_base.xacro (robot description, xacro)
@@ -101,5 +101,5 @@
       <geometry>
         <xacro:if value="${use_mesh_file}">
-          <mesh filename="${mesh_file}" scale="0.002 0.002 0.002" />
+          <mesh filename="${mesh_file}" scale="0.02 0.02 0.02" />
         </xacro:if>
         <xacro:unless value="${use_mesh_file}">
@@ -137,5 +137,5 @@
     image_topic="chase/rgb"
     image_camera_info_topic="chase/camera_info">
-    <origin xyz="-${1.1*body_length} 0 ${0.8*body_height}"/>
+    <origin xyz="-${20*body_length} 0 ${10*body_height}"/>
   </xacro:simple_camera>
   <!-- Color -->
