Commit message: Experimenting with multi agent stuff

File: fcu_sim/urdf/Millennium_Falcon/Millennium_Falcon_base.xacro (robot description, xacro)
@@ -2,7 +2,7 @@
 <robot name="Millennium_Falcon" xmlns:xacro="http://ros.org/wiki/xacro">
   <!-- Properties -->
-  <xacro:property name="namespace" value="Millennium_Falcon"/>
+  <xacro:property name="namespace" value="goldleader"/>
   <xacro:property name="wind_speed_topic" value="gazebo/wind_speed"/>
-  <xacro:property name="command_topic" value="/command"/>
+  <xacro:property name="command_topic" value="command"/>
   <xacro:property name="use_mesh_file" value="true" />
   <xacro:property name="mesh_file" value="package://fcu_sim/meshes/Millennium_Falcon.dae"/>
@@ -98,5 +98,5 @@
     </inertial>
     <visual name="plane_visual">
-      <origin xyz="25 13 -3" rpy="1.570796 0 2.125" />
+      <origin xyz="0 0 0" rpy="0.0 0 1.57295" />
       <geometry>
         <xacro:if value="${use_mesh_file}">

File: fcu_sim/urdf/snowspeeder/snowspeeder_base.xacro (robot description, xacro)
@@ -2,7 +2,7 @@
 <robot name="snowspeeder" xmlns:xacro="http://ros.org/wiki/xacro">
   <!-- Properties -->
-  <xacro:property name="namespace" value="snowspeeder"/>
+  <xacro:property name="namespace" value="rogue1"/>
   <xacro:property name="wind_speed_topic" value="gazebo/wind_speed"/>
-  <xacro:property name="command_topic" value="/command"/>
+  <xacro:property name="command_topic" value="command"/>
   <xacro:property name="use_mesh_file" value="true" />
   <xacro:property name="mesh_file" value="package://fcu_sim/meshes/snowspeeder.dae"/>
